Commit message: updating readme

File: catkin_ws/src/robot_description/urdf/car.urdf (robot description, URDF)
Before this commit: robot car, 8 links, 7 joints
Joints:
- removed joint base_link_to_left_front_steering
- removed joint base_link_to_right_front_steering
- removed joint body_to_left_rear_wheel
- removed joint body_to_right_rear_wheel
- removed joint left_front_steering_to_left_front_wheel
- removed joint right_front_steering_to_right_front_wheel
- added joint left_front_wheel: type continuous, parent left_front_steering, child left_front_wheel, origin xyz=0.0 0.0 0.0, axis 0 1 0
- added joint left_rear_wheel: type continuous, parent body, child left_rear_wheel, origin xyz=0 0.079 0.0, axis 0 1 0
- added joint left_steering: type revolute, parent base_link, child left_front_steering, origin xyz=0.28 0.079 0.054, axis 0 0 1, limit lower=-0.87 upper=0.87 effort=1000 velocity=1000
- added joint right_front_wheel: type continuous, parent right_front_steering, child right_front_wheel, origin xyz=0.0 0.0 0.0, axis 0 1 0
- added joint right_rear_wheel: type continuous, parent body, child right_rear_wheel, origin xyz=0 -0.08 0.0, axis 0 1 0
- added joint right_steering: type revolute, parent base_link, child right_front_steering, origin xyz=0.28 -0.08 0.054, axis 0 0 1, limit lower=-0.87 upper=0.87 effort=1000 velocity=1000

Commit message: Correcting wheels position in urdf, adding interials, collisions and gazebo integration, rear wheels missing

File: catkin_ws/src/robot_description/urdf/car.urdf (robot description, URDF)
Before this commit: robot car, 8 links, 7 joints
Links:
- link base_link: geometry collision box size=0.001 0.001 0.001; visual box size=.001 .001 .001
- link body: mass None -> 2.5; geometry collision box size=0.45 0.2 0.15; visual mesh filename=package://robot_description/models/car_robot/meshes/car.dae
- link left_front_steering: mass None -> 0.001; geometry collision cylinder length=0.025 radius=0.035; visual box size=.001 .001 .001
- link left_front_wheel: mass None -> 0.001; geometry collision cylinder length=0.025 radius=0.035; visual mesh filename=package://robot_description/models/car_robot/meshes/wheel.d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
- link right_front_steering: mass None -> 0.001; geometry collision cylinder length=0.025 radius=0.035; visual box size=.001 .001 .001
- link right_front_wheel: mass None -> 0.001; geometry collision cylinder length=0.025 radius=0.035; visual mesh filename=package://robot_description/models/car_robot/meshes/wheel.d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
Joints:
- removed joint left_front_wheel
- removed joint right_front_wheel
- added joint left_front_wheel_joint: type continuous, parent left_front_steering, child left_front_wheel, origin xyz=0.0 0.0 0.0, axis 0 1 0
- added joint right_front_wheel_joint: type continuous, parent right_front_steering, child right_front_wheel, origin xyz=0.0 0.0 0.0, axis 0 1 0
- joint base_link_to_body: origin xyz=0 0 0.054 -> xyz=0 0 0.0325
- joint left_steering: origin xyz=0.28 0.079 0.054 -> xyz=0.28 0.079 0.0325
- joint right_steering: origin xyz=0.28 -0.08 0.054 -> xyz=0.28 -0.08 0.0325

Commit message: Updating readme and configs

File: catkin_ws/src/robot_description/urdf/car.urdf (robot description, URDF)
Before this commit: robot car, 8 links, 7 joints
Links:
- link left_rear_wheel: mass None -> 0.001; geometry collision cylinder length=0.025 radius=0.035; visual mesh filename=package://robot_description/models/car_robot/meshes/wheel.d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
- link right_rear_wheel: mass None -> 0.001; geometry collision cylinder length=0.025 radius=0.035; visual mesh filename=package://robot_description/models/car_robot/meshes/wheel.d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
Joints:
- removed joint left_rear_wheel
- removed joint right_rear_wheel
- added joint left_rear_wheel_joint: type continuous, parent body, child left_rear_wheel, origin xyz=0 0.079 0.0, axis 0 1 0
- added joint right_rear_wheel_joint: type continuous, parent body, child right_rear_wheel, origin xyz=0 -0.08 0.0, axis 0 1 0
