Commit message: Fixing drifting issue

File: robot_description/urdf/wheel.xacro (robot description, xacro)
@@ -169,4 +169,6 @@
     </gazebo>
     <gazebo reference="${name}_wheel_link">
+      <kp>1e15</kp>
+      <kd>1e13</kd>
     </gazebo>
   </xacro:macro>
@@ -211,4 +213,6 @@
     </transmission>
     <gazebo reference="${name}_wheel_link">
+      <kp>1e15</kp>
+      <kd>1e13</kd>
     </gazebo>
   </xacro:macro>
@@ -299,5 +303,4 @@
     </joint>
     <gazebo reference="${name}_wheel_link">
-      <material>Gazebo/Yellow</material>
     </gazebo>
     <gazebo reference="${name}_wheel_joint">
