Commit message: fix(?) tilted inertia

File: robot_description/urdf/_d435i.urdf.xacro (robot description, xacro)
@@ -49,5 +49,5 @@
   	camera tripod mount -->
     <xacro:property name="d435i_cam_depth_px" value="${d435i_cam_mount_from_center_offset}"/>
-    <xacro:property name="d435i_cam_depth_py" value="0.0175"/>
+    <xacro:property name="d435i_cam_depth_py" value="0.0"/>
     <xacro:property name="d435i_cam_depth_pz" value="${d435i_cam_height/2}"/>
     <material name="${name}_aluminum">
