Commit message: fix broken alignment between laser mesh and lidar link visualizaton

File: robot_description/urdf/lidar.xacro (robot description, xacro)
@@ -4,5 +4,5 @@
     <joint name="hokuyo_joint" type="fixed">
       <axis xyz="0 1 0" />
-      <origin xyz="-0.01 0 0.18" rpy="0 0 0"/>
+      <origin xyz="-0.07 0 0.18" rpy="0 0 0"/>
       <parent link="${parent}"/>
       <child link="car/hokuyo_link"/>
@@ -17,5 +17,5 @@
       </collision>
       <visual>
-        <origin xyz="-0.06 0 -0.03" rpy="0 0 0"/>
+        <origin xyz="0 0 -0.03" rpy="0 0 0"/>
         <geometry>
           <mesh filename="package://robot_description/models/car_robot/meshes/ydlidar.dae"/>
@@ -32,5 +32,5 @@
       <sensor type="ray" name="head_hokuyo_sensor">
         <pose>0 0 0 0 0 0</pose>
-        <visualize>false</visualize>
+        <visualize>true</visualize>
         <update_rate>40</update_rate>
         <ray>
